File: SMCSKart-Mainboard.kicad_sch (KiCad schematic)
At the start: 83 parts, among them J1 Raspberry_Pi_4, J2 Core, J3 MCP4275_Breakout, J4 0430450400, J5 TRANCIEVER, J6 RGB_LED, J7 CAMERA, J8 POWER, J9 MPU-6050_Breakout, Q1 IRLZ44N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

Commit message: update kicad + document connector pinouts
Parts:
- SPARKFUN-GPS-1: value ~ -> (none)
